File: PCB/OlyU-Big/KiCAD/OlyU-Big.kicad_pcb (KiCad board)
At the start: 2 copper layers, 28.5 x 13 mm, 5 parts, among them J1 USB_C_Receptacle, J2 Conn_01x06, J3 Conn_01x02

Commit message: v1.1 update
finalizing data placement and silkscreens
Parts:
- moved J3 1.00 mm to (-6.77, 3.73)
Connections:
- J3 pad 1: D- -> D+
- J3 pad 2: D+ -> D-
Routing:
- net D-: track 21.0 -> 13.8 mm, vias 2 -> 1
- net D+: track 20.2 -> 23.9 mm
- net D3V: track 51.0 -> 54.7 mm
Other:
- board text added: "OlyU-Big"
- board text removed: "OlyU-OEM"
