File: PCB/OlyU-Small/KiCAD/OlyU_v2.kicad_pcb (KiCad board)
At the start: 2 copper layers, 28.4 x 10 mm, 5 parts, among them J1 USB_C_Receptacle, J2 Conn_01x06, J3 Conn_01x02

Commit message: v1.1 update
finalizing data placement and silkscreens
Parts:
- moved J3 1.00 mm to (-6.77, 5.73)
Routing:
- net Net-(J1-PadB5): track 28.6 -> 30.0 mm
- net D3V: track 21.8 -> 22.4 mm
- net GND: track 48.9 -> 49.5 mm
Other:
- board text added: "+"
- board text added: "-"
- board text added: "OlyU"
